Commit message: adding 2

File: install/new_pkg/share/new_pkg/urdf/camera.xacro (robot description, xacro)
@@ -1 +1,58 @@
-/home/ahmad/ros_wc/src/new_pkg/urdf/camera.xacro
+<?xml version='1.0' encoding='utf-8'?>
+<robot name="robot">
+    <link name="camera">
+        <inertial>
+            <origin xyz="0.0 -1.167355140468276e-13 0.0030581760585232944" rpy="0.0 -0.0 0.0" />
+            <mass value="0.02761393779133511" />
+            <inertia ixx="1.4229288925050702e-06" iyy="1.422928887528528e-06" izz="2.5938721415465975e-06" ixy="1.394440118934782e-21" iyz="-1.7954610095097166e-18" ixz="0.0" />
+        </inertial>
+        <visual name="camera_visual">
+            <origin xyz="-0.05 0.0 -0.1" rpy="-3.141592653589793 -1.5707963267948966 0" />
+            <geometry>
+                <mesh filename="file://$(find new_pkg)/meshes/camera.stl" scale="0.001 0.001 0.001" />
+            </geometry>
+            <material name='black'>
+            </material>
+        </visual>
+        <collision name="camera_collision">
+            <origin xyz="-0.05 0.0 -0.1" rpy="-3.141592653589793 -1.5707963267948966 0" />
+            <geometry>
+                <mesh filename="file://$(find new_pkg)/meshes/camera.stl" scale="0.001 0.001 0.001" />
+            </geometry>
+        </collision>
+    </link>
+    <joint name="base_link_Rigid-4" type="fixed">
+        <origin xyz="0.1 0.0 0.05" rpy="-3.141592653589793 -1.5707963267948966 0" />
+        <parent link="base_link" />
+        <child link="camera" />
+    </joint>
+    <link name="camera_link_optical"></link>
+    <joint name="camera_optical_joint" type="fixed">
+        <parent link="camera"/>
+        <child link="camera_link_optical"/>
+        <origin xyz="0 0 0" rpy="${pi} ${-pi/2} 0"/>
+    </joint>
+    <gazebo reference="camera_link_optical">
+        <material>Gazebo/Black</material>
+        <sensor name="camera" type="camera">
+            <pose> 0 0 0 0 0 0 </pose>
+            <visualize>true</visualize>
+            <update_rate>10</update_rate>
+            <camera>
+                <horizontal_fov>1.089</horizontal_fov>
+                <image>
+                    <format>R8G8B8</format>
+                    <width>640</width>
+                    <height>480</height>
+                </image>
+                <clip>
+                    <near>0.05</near>
+                    <far>8.0</far>
+                </clip>
+            </camera>
+            <plugin name="camera_controller" filename="libgazebo_ros_camera.so">
+                <frame_name>camera_link_optical</frame_name>
+            </plugin>
+        </sensor>
+    </gazebo>
+</robot>

File: install/new_pkg/share/new_pkg/urdf/gazebo_cont.xacro (robot description, xacro)
@@ -1 +1,21 @@
-/home/ahmad/ros_wc/src/new_pkg/urdf/gazebo_cont.xacro
+<?xml version="1.0"?>
+<robot xmlns:xacro="http://www.ros.org/wiki/xacro">
+    <gazebo>
+        <plugin name="diff_drive" filename="libgazebo_ros_diff_drive.so">
+            <!-- Wheel Information -->
+            <left_joint>base_link_Revolute-1</left_joint>
+            <right_joint>base_link_Revolute-2</right_joint>
+            <wheel_separation>0.225</wheel_separation>
+            <wheel_diameter>0.1</wheel_diameter>
+            <!-- Limits -->
+            <max_wheel_torque>200</max_wheel_torque>
+            <max_wheel_acceleration>10.0</max_wheel_acceleration>
+            <!-- Output -->
+            <odometry_frame>odom</odometry_frame>
+            <robot_base_frame>base_link</robot_base_frame>
+            <publish_odom>true</publish_odom>
+            <publish_odom_tf>true</publish_odom_tf>
+            <publish_wheel_tf>true</publish_wheel_tf>
+        </plugin>
+    </gazebo>
+</robot>

File: install/new_pkg/share/new_pkg/urdf/lidar.xacro (robot description, xacro)
@@ -1 +1,57 @@
-/home/ahmad/ros_wc/src/new_pkg/urdf/lidar.xacro
+<?xml version='1.0' encoding='utf-8'?>
+<robot name="robot">
+    <link name="lidar">
+        <inertial>
+            <origin xyz="0.0 0.0 0.009999999999999983" rpy="0.0 -0.0 0.0" />
+            <mass value="0.06042068071016568" />
+            <inertia ixx="0.0002051785615782651" iyy="0.0002051785615782755" izz="0.0003700766693497588" ixy="-8.924416761146858e-20" iyz="-4.908429218630772e-19" ixz="-4.336808689942018e-19" />
+        </inertial>
+        <visual name="lidar_visual">
+            <origin xyz="-0.05 0.0 -0.1" rpy="0.0 -0.0 0.0" />
+            <geometry>
+                <mesh filename="file://$(find new_pkg)/meshes/lidar.stl" scale="0.001 0.001 0.001" />
+            </geometry>
+            <material name='black'>
+            </material>
+        </visual>
+        <collision name="lidar_collision">
+            <origin xyz="-0.05 0.0 -0.1" rpy="0.0 -0.0 0.0" />
+            <geometry>
+                <mesh filename="file://$(find new_pkg)/meshes/lidar.stl" scale="0.001 0.001 0.001" />
+            </geometry>
+        </collision>
+    </link>
+    <joint name="base_link_Rigid-3" type="fixed">
+        <origin xyz="0.05 0.0 0.1" rpy="0.0 -0.0 0.0" />
+        <parent link="base_link" />
+        <child link="lidar" />
+    </joint>
+    <gazebo reference="lidar">
+        <material>Gazebo/Black</material>
+        <sensor name="laser" type="ray">
+            <pose> 0 0 0 0 0 0 </pose>
+            <visualize>true</visualize>
+            <update_rate>10</update_rate>
+            <ray>
+                <scan>
+                    <horizontal>
+                        <samples>360</samples>
+                        <min_angle>-3.14</min_angle>
+                        <max_angle>3.14</max_angle>
+                    </horizontal>
+                </scan>
+                <range>
+                    <min>0.3</min>
+                    <max>12</max>
+                </range>
+            </ray>
+            <plugin name="laser_controller" filename="libgazebo_ros_ray_sensor.so">
+                <ros>
+                    <argument>~/out:=scan</argument>
+                </ros>
+                <output_type>sensor_msgs/LaserScan</output_type>
+                <frame_name>lidar</frame_name>
+            </plugin>
+        </sensor>
+    </gazebo>
+</robot>

File: install/new_pkg/share/new_pkg/urdf/robot.urdf.xacro (robot description, xacro)
@@ -1 +1,7 @@
-/home/ahmad/ros_wc/src/new_pkg/urdf/robot.urdf.xacro
+<?xml version="1.0"?>
+<robot xmlns:xacro="http://www.ros.org/wiki/xacro"  name="robot">
+    <xacro:include filename="robot_body.xacro" />
+    <xacro:include filename="camera.xacro" />
+    <xacro:include filename="lidar.xacro" />
+    <xacro:include filename="gazebo_cont.xacro" />
+</robot>

File: install/new_pkg/share/new_pkg/urdf/robot_body.xacro (robot description, xacro)
@@ -1 +1,95 @@
-/home/ahmad/ros_wc/src/new_pkg/urdf/robot_body.xacro
+<?xml version='1.0' encoding='utf-8'?>
+<robot name="robot">
+    <material name='white'>
+        <color rgba="1.0 1.0 1.0 1.0"/>
+    </material>
+    <material name='black'>
+        <color rgba="0.0 0.0 0.0 1.0"/>
+    </material>
+    <link name="base_link">
+        <inertial>
+            <origin xyz="0.0038662210655893464 0.0 0.052675337982169175" rpy="0.0 0.0 0.0" />
+            <mass value="1.713155401009962" />
+            <inertia ixx="0.0584527227543141" iyy="0.06191909363698124" izz="0.10992638017861338" ixy="0.0" iyz="0.0" ixz="-0.002306589723332078" />
+        </inertial>
+        <visual name="base_link_visual">
+            <origin xyz="0.0 0.0 0.0" rpy="0.0 0.0 0.0" />
+            <geometry>
+                <mesh filename="file://$(find new_pkg)/meshes/base_link.stl" scale="0.001 0.001 0.001" />
+            </geometry>
+            <material name='white'>
+            </material>
+        </visual>
+        <collision name="base_link_collision">
+            <origin xyz="0.0 0.0 0.0" rpy="0.0 0.0 0.0" />
+            <geometry>
+                <mesh filename="file://$(find new_pkg)/meshes/base_link.stl" scale="0.001 0.001 0.001" />
+            </geometry>
+        </collision>
+    </link>
+    <gazebo reference="base_link">
+        <material>Gazebo/White</material>
+        <mu1 value="0.001"/>
+        <mu2 value="0.001"/>
+    </gazebo>
+    <link name="right_wheel">
+        <inertial>
+            <origin xyz="5.7900231001220315e-18 0.0 0.012500000000000053" rpy="0.0 -0.0 0.0" />
+            <mass value="0.15413438956674914" />
+            <inertia ixx="0.0010436182626914897" iyy="0.0010436182626915452" izz="0.0019266798695843383" ixy="2.677325028344055e-19" iyz="1.734723475976807e-18" ixz="-1.7179502265207697e-18" />
+        </inertial>
+        <visual name="right_wheel_visual">
+            <origin xyz="0.0 0.05 0.12500000000000003" rpy="1.5707963267948966 -0.0 0.0" />
+            <geometry>
+                <mesh filename="file://$(find new_pkg)/meshes/right_wheel.stl" scale="0.001 0.001 0.001" />
+            </geometry>
+            <material name='black'>
+            </material>
+        </visual>
+        <collision name="right_wheel_collision">
+            <origin xyz="0.0 0.05 0.12500000000000003" rpy="1.5707963267948966 -0.0 0.0" />
+            <geometry>
+                <mesh filename="file://$(find new_pkg)/meshes/right_wheel.stl" scale="0.001 0.001 0.001" />
+            </geometry>
+        </collision>
+    </link>
+    <gazebo reference="right_wheel">
+        <material>Gazebo/Black</material>
+    </gazebo>
+    <link name="left_wheel">
+        <inertial>
+            <origin xyz="5.7900231001220315e-18 0.0 0.012500000000000018" rpy="0.0 -0.0 0.0" />
+            <mass value="0.15413438956674914" />
+            <inertia ixx="0.0010436182626914932" iyy="0.0010436182626915522" izz="0.0019266798695843383" ixy="2.677325028344058e-19" iyz="0.0" ixz="1.5394618912978329e-18" />
+        </inertial>
+        <visual name="left_wheel_visual">
+            <origin xyz="0.0 0.05 -0.1" rpy="1.5707963267948966 -0.0 0.0" />
+            <geometry>
+                <mesh filename="file://$(find new_pkg)/meshes/left_wheel.stl" scale="0.001 0.001 0.001" />
+            </geometry>
+            <material name='black'>
+            </material>
+        </visual>
+        <collision name="left_wheel_collision">
+            <origin xyz="0.0 0.05 -0.1" rpy="1.5707963267948966 -0.0 0.0" />
+            <geometry>
+                <mesh filename="file://$(find new_pkg)/meshes/left_wheel.stl" scale="0.001 0.001 0.001" />
+            </geometry>
+        </collision>
+    </link>
+    <gazebo reference="left_wheel">
+        <material>Gazebo/Black</material>
+    </gazebo>
+    <joint name="base_link_Revolute-1" type="continuous">
+        <origin xyz="0.0 0.1 0.05" rpy="-1.5707963267948966 -0.0 0.0" />
+        <parent link="base_link" />
+        <child link="left_wheel" />
+        <axis xyz="0.0 0.0 1.0" />
+    </joint>
+    <joint name="base_link_Revolute-2" type="continuous">
+        <origin xyz="0.0 -0.1 0.05" rpy="1.5707963267948966 -0.0 0.0" />
+        <parent link="base_link" />
+        <child link="right_wheel" />
+        <axis xyz="0.0 0.0 -1.0" />
+    </joint>
+</robot>

File: src/new_pkg/urdf/camera.xacro (robot description, xacro)
@@ -1,47 +1,58 @@
 <?xml version='1.0' encoding='utf-8'?>
 <robot name="robot">
-<link name="camera">
-    <inertial>
-        <origin xyz="0.0 -1.167355140468276e-13 0.0030581760585232944" rpy="0.0 -0.0 0.0" />
-        <mass value="0.02761393779133511" />
-        <inertia ixx="1.4229288925050702e-06" iyy="1.422928887528528e-06" izz="2.5938721415465975e-06" ixy="1.394440118934782e-21" iyz="-1.7954610095097166e-18" ixz="0.0" />
-    </inertial>
-    <visual name="camera_visual">
-        <origin xyz="-0.05 0.0 -0.1" rpy="-3.141592653589793 -1.5707963267948966 0" />
-        <geometry>
-            <mesh filename="file://$(find new_pkg)/meshes/camera.stl" scale="0.001 0.001 0.001" />
-        </geometry>
-        <material name="black">
-        </material>
-    </visual>
-    <collision name="camera_collision">
-        <origin xyz="-0.05 0.0 -0.1" rpy="-3.141592653589793 -1.5707963267948966 0" />
-        <geometry>
-            <mesh filename="file://$(find new_pkg)/meshes/camera.stl" scale="0.001 0.001 0.001" />
-        </geometry>
-    </collision>
-</link>
-<gazebo reference="camera">
-    <material>Gazebo/Black</material>
-    <sensor name="camera" type="camera">
-        <pose> 0 0 0 0 0 0 </pose>
-        <visualize>true</visualize>
-        <update_rate>10</update_rate>
-        <camera>
-            <horizontal_fov>1.089</horizontal_fov>
-            <image>
-                <format>R8G8B8</format>
-                <width>640</width>
-                <height>480</height>
-            </image>
-            <clip>
-                <near>0.05</near>
-                <far>8.0</far>
-            </clip>
-        </camera>
-        <plugin name="camera_controller" filename="libgazebo_ros_camera.so">
-            <frame_name>camera</frame_name>
-        </plugin>
-    </sensor>
-</gazebo>
+    <link name="camera">
+        <inertial>
+            <origin xyz="0.0 -1.167355140468276e-13 0.0030581760585232944" rpy="0.0 -0.0 0.0" />
+            <mass value="0.02761393779133511" />
+            <inertia ixx="1.4229288925050702e-06" iyy="1.422928887528528e-06" izz="2.5938721415465975e-06" ixy="1.394440118934782e-21" iyz="-1.7954610095097166e-18" ixz="0.0" />
+        </inertial>
+        <visual name="camera_visual">
+            <origin xyz="-0.05 0.0 -0.1" rpy="-3.141592653589793 -1.5707963267948966 0" />
+            <geometry>
+                <mesh filename="file://$(find new_pkg)/meshes/camera.stl" scale="0.001 0.001 0.001" />
+            </geometry>
+            <material name='black'>
+            </material>
+        </visual>
+        <collision name="camera_collision">
+            <origin xyz="-0.05 0.0 -0.1" rpy="-3.141592653589793 -1.5707963267948966 0" />
+            <geometry>
+                <mesh filename="file://$(find new_pkg)/meshes/camera.stl" scale="0.001 0.001 0.001" />
+            </geometry>
+        </collision>
+    </link>
+    <joint name="base_link_Rigid-4" type="fixed">
+        <origin xyz="0.1 0.0 0.05" rpy="-3.141592653589793 -1.5707963267948966 0" />
+        <parent link="base_link" />
+        <child link="camera" />
+    </joint>
+    <link name="camera_link_optical"></link>
+    <joint name="camera_optical_joint" type="fixed">
+        <parent link="camera"/>
+        <child link="camera_link_optical"/>
+        <origin xyz="0 0 0" rpy="${pi} ${-pi/2} 0"/>
+    </joint>
+    <gazebo reference="camera_link_optical">
+        <material>Gazebo/Black</material>
+        <sensor name="camera" type="camera">
+            <pose> 0 0 0 0 0 0 </pose>
+            <visualize>true</visualize>
+            <update_rate>10</update_rate>
+            <camera>
+                <horizontal_fov>1.089</horizontal_fov>
+                <image>
+                    <format>R8G8B8</format>
+                    <width>640</width>
+                    <height>480</height>
+                </image>
+                <clip>
+                    <near>0.05</near>
+                    <far>8.0</far>
+                </clip>
+            </camera>
+            <plugin name="camera_controller" filename="libgazebo_ros_camera.so">
+                <frame_name>camera_link_optical</frame_name>
+            </plugin>
+        </sensor>
+    </gazebo>
 </robot>

File: src/new_pkg/urdf/lidar.xacro (robot description, xacro)
@@ -1,52 +1,57 @@
 <?xml version='1.0' encoding='utf-8'?>
 <robot name="robot">
-<link name="lidar">
-    <inertial>
-        <origin xyz="0.0 0.0 0.009999999999999983" rpy="0.0 -0.0 0.0" />
-        <mass value="0.6042068071016568" />
-        <inertia ixx="0.0002051785615782651" iyy="0.0002051785615782755" izz="0.0003700766693497588" ixy="-8.924416761146858e-20" iyz="-4.908429218630772e-19" ixz="-4.336808689942018e-19" />
-    </inertial>
-    <visual name="lidar_visual">
-        <origin xyz="-0.05 0.0 -0.1" rpy="0.0 -0.0 0.0" />
-        <geometry>
-            <mesh filename="file://$(find new_pkg)/meshes/lidar.stl" scale="0.001 0.001 0.001" />
-        </geometry>
-        <material name="black">
-        </material>
-    </visual>
-    <collision name="lidar_collision">
-        <origin xyz="-0.05 0.0 -0.1" rpy="0.0 -0.0 0.0" />
-        <geometry>
-            <mesh filename="file://$(find new_pkg)/meshes/lidar.stl" scale="0.001 0.001 0.001" />
-        </geometry>
-    </collision>
-</link>
-<gazebo reference="lidar">
-    <material>Gazebo/Black</material>
-    <sensor name="laser" type="ray">
-        <pose> 0 0 0 0 0 0 </pose>
-        <visualize>true</visualize>
-        <update_rate>10</update_rate>
-        <ray>
-            <scan>
-                <horizontal>
-                    <samples>360</samples>
-                    <min_angle>-3.14</min_angle>
-                    <max_angle>3.14</max_angle>
-                </horizontal>
-            </scan>
-            <range>
-                <min>0.3</min>
-                <max>12</max>
-            </range>
-        </ray>
-        <plugin name="laser_controller" filename="libgazebo_ros_ray_sensor.so">
-            <ros>
-                <argument>~/out:=scan</argument>
-            </ros>
-            <output_type>sensor_msgs/LaserScan</output_type>
-            <frame_name>lidar</frame_name>
-        </plugin>
-    </sensor>
-</gazebo>
+    <link name="lidar">
+        <inertial>
+            <origin xyz="0.0 0.0 0.009999999999999983" rpy="0.0 -0.0 0.0" />
+            <mass value="0.06042068071016568" />
+            <inertia ixx="0.0002051785615782651" iyy="0.0002051785615782755" izz="0.0003700766693497588" ixy="-8.924416761146858e-20" iyz="-4.908429218630772e-19" ixz="-4.336808689942018e-19" />
+        </inertial>
+        <visual name="lidar_visual">
+            <origin xyz="-0.05 0.0 -0.1" rpy="0.0 -0.0 0.0" />
+            <geometry>
+                <mesh filename="file://$(find new_pkg)/meshes/lidar.stl" scale="0.001 0.001 0.001" />
+            </geometry>
+            <material name='black'>
+            </material>
+        </visual>
+        <collision name="lidar_collision">
+            <origin xyz="-0.05 0.0 -0.1" rpy="0.0 -0.0 0.0" />
+            <geometry>
+                <mesh filename="file://$(find new_pkg)/meshes/lidar.stl" scale="0.001 0.001 0.001" />
+            </geometry>
+        </collision>
+    </link>
+    <joint name="base_link_Rigid-3" type="fixed">
+        <origin xyz="0.05 0.0 0.1" rpy="0.0 -0.0 0.0" />
+        <parent link="base_link" />
+        <child link="lidar" />
+    </joint>
+    <gazebo reference="lidar">
+        <material>Gazebo/Black</material>
+        <sensor name="laser" type="ray">
+            <pose> 0 0 0 0 0 0 </pose>
+            <visualize>true</visualize>
+            <update_rate>10</update_rate>
+            <ray>
+                <scan>
+                    <horizontal>
+                        <samples>360</samples>
+                        <min_angle>-3.14</min_angle>
+                        <max_angle>3.14</max_angle>
+                    </horizontal>
+                </scan>
+                <range>
+                    <min>0.3</min>
+                    <max>12</max>
+                </range>
+            </ray>
+            <plugin name="laser_controller" filename="libgazebo_ros_ray_sensor.so">
+                <ros>
+                    <argument>~/out:=scan</argument>
+                </ros>
+                <output_type>sensor_msgs/LaserScan</output_type>
+                <frame_name>lidar</frame_name>
+            </plugin>
+        </sensor>
+    </gazebo>
 </robot>

File: src/new_pkg/urdf/robot.urdf.xacro (robot description, xacro)
@@ -2,6 +2,6 @@
 <robot xmlns:xacro="http://www.ros.org/wiki/xacro"  name="robot">
     <xacro:include filename="robot_body.xacro" />
+    <xacro:include filename="camera.xacro" />
+    <xacro:include filename="lidar.xacro" />
     <xacro:include filename="gazebo_cont.xacro" />
-    <xacro:include filename="lidar.xacro" />
-    <xacro:include filename="camera.xacro" />
 </robot>

File: src/new_pkg/urdf/robot_body.xacro (robot description, xacro)
@@ -1,8 +1,8 @@
 <?xml version='1.0' encoding='utf-8'?>
 <robot name="robot">
-    <material name="white">
+    <material name='white'>
         <color rgba="1.0 1.0 1.0 1.0"/>
     </material>
-    <material name="black">
+    <material name='black'>
         <color rgba="0.0 0.0 0.0 1.0"/>
     </material>
@@ -18,5 +18,5 @@
                 <mesh filename="file://$(find new_pkg)/meshes/base_link.stl" scale="0.001 0.001 0.001" />
             </geometry>
-            <material name="white">
+            <material name='white'>
             </material>
         </visual>
@@ -29,7 +29,7 @@
     </link>
     <gazebo reference="base_link">
-         <material>Gazebo/Black</material>
-         <mu1 value="0.001"/>
-         <mu2 value="0.001"/>
+        <material>Gazebo/White</material>
+        <mu1 value="0.001"/>
+        <mu2 value="0.001"/>
     </gazebo>
     <link name="right_wheel">
@@ -44,5 +44,5 @@
                 <mesh filename="file://$(find new_pkg)/meshes/right_wheel.stl" scale="0.001 0.001 0.001" />
             </geometry>
-            <material name="black">
+            <material name='black'>
             </material>
         </visual>
@@ -55,6 +55,6 @@
     </link>
     <gazebo reference="right_wheel">
-        <material>Gazebo/White</material>
-   </gazebo>
+        <material>Gazebo/Black</material>
+    </gazebo>
     <link name="left_wheel">
         <inertial>
@@ -68,5 +68,5 @@
                 <mesh filename="file://$(find new_pkg)/meshes/left_wheel.stl" scale="0.001 0.001 0.001" />
             </geometry>
-            <material name="black">
+            <material name='black'>
             </material>
         </visual>
@@ -79,6 +79,6 @@
     </link>
     <gazebo reference="left_wheel">
-        <material>Gazebo/White</material>
-   </gazebo>
+        <material>Gazebo/Black</material>
+    </gazebo>
     <joint name="base_link_Revolute-1" type="continuous">
         <origin xyz="0.0 0.1 0.05" rpy="-1.5707963267948966 -0.0 0.0" />
@@ -93,13 +93,3 @@
         <axis xyz="0.0 0.0 -1.0" />
     </joint>
-    <joint name="base_link_Rigid-3" type="fixed">
-        <origin xyz="0.05 0.0 0.1" rpy="0.0 -0.0 0.0" />
-        <parent link="base_link" />
-        <child link="lidar" />
-    </joint>
-    <joint name="base_link_Rigid-4" type="fixed">
-        <origin xyz="0.1 0.0 0.05" rpy="-3.141592653589793 -1.5707963267948966 0" />
-        <parent link="base_link" />
-        <child link="camera" />
-    </joint>
 </robot>
